File: hardware/dual-relay.kicad_pcb (KiCad board)
At the start: 2 copper layers, 40 x 40 mm, 34 parts, among them P1 CON-SENSOR2, P2 BOOT, P3 CONN_8, P4 Debug, Q1 SSM6N7002KFU, U1 XMC1XXX24, U2 G5LE-1-36, U3 G5LE-1-36, U4 DRILL, U5 DRILL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

Commit message: specify processor
Parts:
- U1: value XMC1XXX24 -> XMC1100
Changed lines of the file:
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@@
       (effects (font (size 0.3 0.3) (thickness 0.075)))
     )
-    (fp_text value XMC1XXX24 (at 0 0.8 135) (layer F.Fab)
+    (fp_text value XMC1100 (at 0 0.8 135) (layer F.Fab)
       (effects (font (size 0.3 0.3) (thickness 0.075)))
     )
@@
   (gr_line (start 136.075 109.475) (end 133.675 109.475) (angle 90) (layer B.SilkS) (width 0.381))
   (gr_line (start 135.5 112.975) (end 134.15 114.325) (angle 90) (layer B.SilkS) (width 0.381))
-  (gr_text Status (at 167.575 112.675 -90) (layer F.SilkS)
+  (gr_text Status (at 167.575 112.675 270) (layer F.SilkS)
     (effects (font (size 0.7 0.7) (thickness 0.14986)))
   )

Commit message: Add 3d information (final)
Parts:
- U2, U3: footprint G5LE-1 -> kicad-libraries:G5LE-1
Changed lines of the file:
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@@
-(kicad_pcb (version 4) (host pcbnew 4.0.7-e2-6376~58~ubuntu17.04.1)
+(kicad_pcb (version 4) (host pcbnew 4.0.2+dfsg1-stable)
   (general
     (links 61)
     (no_connects 0)
-    (area 131.220139 83.320139 282.19527 165.489573)
+    (area 131.973659 84.071159 172.175001 124.275001)
     (thickness 1.6002)
     (drawings 34)
@@
     )
   )
-  (module G5LE-1 (layer Vorderseite)
-    (at 153.075 115.175 180)
-    (fp_text reference U3 (at 0.1 -2.7 180) (layer F.Fab)
-      (effects (font (size 0.3 0.3) (thickness 0.075)))
-    )
-    (fp_text value G5LE-1-36 (at 0 0 180) (layer F.Fab)
-      (effects (font (size 0.3 0.3) (thickness 0.075)))
-    )
-    (fp_line (start -11.3 -8.3) (end 11.3 -8.3) (layer F.Fab) (width 0.1))
-    (fp_line (start 11.3 -8.3) (end 11.3 8.3) (layer F.Fab) (width 0.1))
-    (fp_line (start 11.3 8.3) (end -11.3 8.3) (layer F.Fab) (width 0.1))
-    (fp_line (start -11.3 8.3) (end -11.3 -8.3) (layer F.Fab) (width 0.1))
-    (pad 1 thru_hole circle (at -6.7 -6 180) (size 2.6 2.6) (drill 1.3) (layers *.Cu *.Mask F.SilkS)
-      (net 1 +5V))
-    (pad 2 thru_hole circle (at -8.7 0 180) (size 2.6 2.6) (drill 1.3) (layers *.Cu *.Mask F.SilkS)
-      (net 25 "Net-(P3-Pad7)"))
-    (pad 3 thru_hole circle (at -6.7 6 180) (size 2.6 2.6) (drill 1.3) (layers *.Cu *.Mask F.SilkS)
-      (net 15 "Net-(D5-Pad1)"))
-    (pad 4 thru_hole circle (at 5.5 6 180) (size 2.6 2.6) (drill 1.3) (layers *.Cu *.Mask F.SilkS)
-      (net 24 "Net-(P3-Pad6)"))
-    (pad 5 thru_hole circle (at 5.5 -6 180) (size 2.6 2.6) (drill 1.3) (layers *.Cu *.Mask F.SilkS)
-      (net 26 "Net-(P3-Pad8)"))
-  )
   (module C0603F (layer Vorderseite)
     (at 165.575 105.375 90)
@@
     )
   )
-  (module G5LE-1 (layer Vorderseite)
-    (at 153.075 93.175 180)
-    (fp_text reference U2 (at 0.1 -2.7 180) (layer F.Fab)
-      (effects (font (size 0.3 0.3) (thickness 0.075)))
-    )
-    (fp_text value G5LE-1-36 (at 0 0 180) (layer F.Fab)
-      (effects (font (size 0.3 0.3) (thickness 0.075)))
-    )
-    (fp_line (start -11.3 -8.3) (end 11.3 -8.3) (layer F.Fab) (width 0.1))
-    (fp_line (start 11.3 -8.3) (end 11.3 8.3) (layer F.Fab) (width 0.1))
-    (fp_line (start 11.3 8.3) (end -11.3 8.3) (layer F.Fab) (width 0.1))
-    (fp_line (start -11.3 8.3) (end -11.3 -8.3) (layer F.Fab) (width 0.1))
-    (pad 1 thru_hole circle (at -6.7 -6 180) (size 2.6 2.6) (drill 1.3) (layers *.Cu *.Mask F.SilkS)
-      (net 1 +5V))
-    (pad 2 thru_hole circle (at -8.7 0 180) (size 2.6 2.6) (drill 1.3) (layers *.Cu *.Mask F.SilkS)
-      (net 21 "Net-(P3-Pad2)"))
-    (pad 3 thru_hole circle (at -6.7 6 180) (size 2.6 2.6) (drill 1.3) (layers *.Cu *.Mask F.SilkS)
-      (net 14 "Net-(D4-Pad1)"))
-    (pad 4 thru_hole circle (at 5.5 6 180) (size 2.6 2.6) (drill 1.3) (layers *.Cu *.Mask F.SilkS)
-      (net 23 "Net-(P3-Pad1)"))
-    (pad 5 thru_hole circle (at 5.5 -6 180) (size 2.6 2.6) (drill 1.3) (layers *.Cu *.Mask F.SilkS)
-      (net 22 "Net-(P3-Pad3)"))
-  )
   (module DRILL_NP (layer Vorderseite)
     (at 169.575 121.675)
@@
     )
   )
+  (module kicad-libraries:G5LE-1 (layer Vorderseite)
+    (at 153.075 93.175 180)
+    (fp_text reference U2 (at 0.1 -2.7 180) (layer F.Fab)
+      (effects (font (size 0.3 0.3) (thickness 0.075)))
+    )
+    (fp_text value G5LE-1-36 (at 0 0 180) (layer F.Fab)
+      (effects (font (size 0.3 0.3) (thickness 0.075)))
+    )
+    (fp_line (start -11.3 -8.3) (end 11.3 -8.3) (layer F.Fab) (width 0.1))
+    (fp_line (start 11.3 -8.3) (end 11.3 8.3) (layer F.Fab) (width 0.1))
+    (fp_line (start 11.3 8.3) (end -11.3 8.3) (layer F.Fab) (width 0.1))
+    (fp_line (start -11.3 8.3) (end -11.3 -8.3) (layer F.Fab) (width 0.1))
+    (pad 1 thru_hole circle (at -6.7 -6 180) (size 2.6 2.6) (drill 1.3) (layers *.Cu *.Mask F.SilkS)
+      (net 1 +5V))
+    (pad 2 thru_hole circle (at -8.7 0 180) (size 2.6 2.6) (drill 1.3) (layers *.Cu *.Mask F.SilkS)
+      (net 21 "Net-(P3-Pad2)"))
+    (pad 3 thru_hole circle (at -6.7 6 180) (size 2.6 2.6) (drill 1.3) (layers *.Cu *.Mask F.SilkS)
+      (net 14 "Net-(D4-Pad1)"))
+    (pad 4 thru_hole circle (at 5.5 6 180) (size 2.6 2.6) (drill 1.3) (layers *.Cu *.Mask F.SilkS)
+      (net 23 "Net-(P3-Pad1)"))
+    (pad 5 thru_hole circle (at 5.5 -6 180) (size 2.6 2.6) (drill 1.3) (layers *.Cu *.Mask F.SilkS)
+      (net 22 "Net-(P3-Pad3)"))
+    (model Buttons_Switches/G5LE-1-Relay.wrl
+      (at (xyz 0 0 0))
+      (scale (xyz 1 1 1))
+      (rotate (xyz 270 0 0))
+    )
+  )
+  (module kicad-libraries:G5LE-1 (layer Vorderseite)
+    (at 153.075 115.175 180)
+    (fp_text reference U3 (at 0.1 -2.7 180) (layer F.Fab)
+      (effects (font (size 0.3 0.3) (thickness 0.075)))
+    )
+    (fp_text value G5LE-1-36 (at 0 0 180) (layer F.Fab)
+      (effects (font (size 0.3 0.3) (thickness 0.075)))
+    )
+    (fp_line (start -11.3 -8.3) (end 11.3 -8.3) (layer F.Fab) (width 0.1))
+    (fp_line (start 11.3 -8.3) (end 11.3 8.3) (layer F.Fab) (width 0.1))
+    (fp_line (start 11.3 8.3) (end -11.3 8.3) (layer F.Fab) (width 0.1))
+    (fp_line (start -11.3 8.3) (end -11.3 -8.3) (layer F.Fab) (width 0.1))
+    (pad 1 thru_hole circle (at -6.7 -6 180) (size 2.6 2.6) (drill 1.3) (layers *.Cu *.Mask F.SilkS)
+      (net 1 +5V))
+    (pad 2 thru_hole circle (at -8.7 0 180) (size 2.6 2.6) (drill 1.3) (layers *.Cu *.Mask F.SilkS)
+      (net 25 "Net-(P3-Pad7)"))
+    (pad 3 thru_hole circle (at -6.7 6 180) (size 2.6 2.6) (drill 1.3) (layers *.Cu *.Mask F.SilkS)
+      (net 15 "Net-(D5-Pad1)"))
+    (pad 4 thru_hole circle (at 5.5 6 180) (size 2.6 2.6) (drill 1.3) (layers *.Cu *.Mask F.SilkS)
+      (net 24 "Net-(P3-Pad6)"))
+    (pad 5 thru_hole circle (at 5.5 -6 180) (size 2.6 2.6) (drill 1.3) (layers *.Cu *.Mask F.SilkS)
+      (net 26 "Net-(P3-Pad8)"))
+    (model Buttons_Switches/G5LE-1-Relay.wrl
+      (at (xyz 0 0 0))
+      (scale (xyz 1 1 1))
+      (rotate (xyz 270 0 0))
+    )
+  )
