File: hardware/industrial-dual-relay.kicad_pcb (KiCad board)
At the start: 2 copper layers, 40 x 40 mm, 34 parts, among them P1 CON-SENSOR2, P2 BOOT, P3 CONN_8, P4 Debug, Q2 G5Q-1, Q3 G5Q-1, U1 XMC1100, U4 DRILL, U5 DRILL, U6 DRILL

Commit message: Data Cleanup
Parts:
- REF**, U4, U5, U6: footprint kicad-libraries:DRILL_NP_New -> kicad-libraries:DRILL_NP
Connections:
- U1 pad 18: RELAY0 -> RELAY1
- U1 pad 19: RELAY1 -> RELAY0
Changed lines of the file:
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@@
     )
   )
-  (footprint "kicad-libraries:DRILL_NP_New" (layer "F.Cu")
+  (footprint "kicad-libraries:DRILL_NP" (layer "F.Cu")
     (at 169.3 86.4 90)
     (fp_text reference "U4" (at 0 -0.5 90 unlocked) (layer "F.Fab")
@@
       (clearance 0.89))
   )
-  (footprint "kicad-libraries:DRILL_NP_New" (layer "F.Cu")
+  (footprint "kicad-libraries:DRILL_NP" (layer "F.Cu")
     (at 169.3 121.4 90)
     (fp_text reference "U5" (at 0 -0.5 90 unlocked) (layer "F.Fab")
@@
       (clearance 0.89))
   )
-  (footprint "kicad-libraries:DRILL_NP_New" (layer "F.Cu")
+  (footprint "kicad-libraries:DRILL_NP" (layer "F.Cu")
     (at 134.3 121.4 90)
     (fp_text reference "U6" (at 0 -0.5 90 unlocked) (layer "F.Fab")
@@
       (net 24 "Net-(P3-Pad6)") (pintype "input"))
   )
-  (footprint "kicad-libraries:DRILL_NP_New" (layer "F.Cu")
+  (footprint "kicad-libraries:DRILL_NP" (layer "F.Cu")
     (at 134.3 86.4)
     (fp_text reference "REF**" (at 0 -0.5 unlocked) (layer "F.Fab")
@@
       (net 40 "unconnected-(U1-Pad17)") (pinfunction "P0.6_IO") (pintype "passive+no_connect"))
     (pad "18" smd oval locked (at 2.025 -1.25 225) (size 1 0.3) (layers "F.Cu" "F.Paste" "F.Mask")
-      (net 9 "RELAY0") (pinfunction "P0.7_IO") (pintype "passive"))
+      (net 8 "RELAY1") (pinfunction "P0.7_IO") (pintype "passive"))
     (pad "19" smd oval locked (at 1.25 -2.025 315) (size 1 0.3) (layers "F.Cu" "F.Paste" "F.Mask")
-      (net 8 "RELAY1") (pinfunction "P0.8_IO") (pintype "passive"))
+      (net 9 "RELAY0") (pinfunction "P0.8_IO") (pintype "passive"))
     (pad "20" smd oval locked (at 0.75 -2.025 315) (size 1 0.3) (layers "F.Cu" "F.Paste" "F.Mask")
       (net 2 "GND") (pinfunction "P0.9_IO") (pintype "passive"))
