File: hardware/industrial-dual-relay.kicad_sch (KiCad schematic)
At the start: 27 parts, among them P1 CON-SENSOR2, P2 BOOT, P3 CONN_8, P4 Debug, Q1 SSM6N7002KFU, Q2 G5Q-1, Q3 G5Q-1, U1 XMC1100, U4 DRILL, U5 DRILL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

Commit message: Data cleanup.
Parts:
- U4, U5, U6, U7: footprint kicad-libraries:DRILL_NP -> kicad-libraries:DRILL_NP_New
Other:
- note added: "Copyright Tinkerforge GmbH 2023. This documentation describes Open Hardware and is licensed under the CERN OHL v. 1.1. You may redistribute and modify this documentation under the terms of the CERN OHL v.1.1. (http://ohwr.org/cernohl). This documentation is distributed WITHOUT ANY EXPRESS OR IMPLIED WARRANTY, INCLUDING OF MERCHANTABILITY, SATISFACTORY QUALITY AND FITNESS FOR A PARTICULAR PURPOSE.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"
- note removed: "Copyright Tinkerforge GmbH 2017. This documentation describes Open Hardware and is licensed under the CERN OHL v. 1.1. You may redistribute and modify this documentation under the terms of the CERN OHL v.1.1. (http://ohwr.org/cernohl). This documentation is distributed WITHOUT ANY EXPRESS OR IMPLIED WARRANTY, INCLUDING OF MERCHANTABILITY, SATISFACTORY QUALITY AND FITNESS FOR A PARTICULAR PURPOSE.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"
Changed lines of the file:
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@@
   (title_block
     (title "Industrial Dual Relay")
-    (date "2017-12-06")
-    (rev "1.0")
+    (date "2023-01-24")
+    (rev "1.2")
     (company "Tinkerforge GmbH")
     (comment 1 "Licensed under CERN OHL v.1.1")
-    (comment 2 "Copyright (©) 2017, B.Nordmeyer <bastian@tinkerforge.com>")
+    (comment 2 "Copyright (©) 2023, B.Nordmeyer <bastian@tinkerforge.com>")
   )
   (junction (at 116.84 173.99) (diameter 0) (color 0 0 0 0)
@@
     (stroke (width 0) (type default) (color 0 0 0 0))
   )
-  (text "Copyright Tinkerforge GmbH 2017.\nThis documentation describes Open Hardware and is licensed under the\nCERN OHL v. 1.1.\nYou may redistribute and modify this documentation under the terms of the\nCERN OHL v.1.1. (http://ohwr.org/cernohl). This documentation is distributed\nWITHOUT ANY EXPRESS OR IMPLIED WARRANTY, INCLUDING OF\nMERCHANTABILITY, SATISFACTORY QUALITY AND FITNESS FOR A\nPARTICULAR PURPOSE. Please see the CERN OHL v.1.1 for applicable\nconditions\n"
+  (text "Copyright Tinkerforge GmbH 2023.\nThis documentation describes Open Hardware and is licensed under the\nCERN OHL v. 1.1.\nYou may redistribute and modify this documentation under the terms of the\nCERN OHL v.1.1. (http://ohwr.org/cernohl). This documentation is distributed\nWITHOUT ANY EXPRESS OR IMPLIED WARRANTY, INCLUDING OF\nMERCHANTABILITY, SATISFACTORY QUALITY AND FITNESS FOR A\nPARTICULAR PURPOSE. Please see the CERN OHL v.1.1 for applicable\nconditions\n"
     (at 13.97 195.58 0)
     (effects (font (size 1.016 1.016)) (justify left bottom))
@@
       (effects (font (size 1.524 1.524)))
     )
-    (property "Footprint" "kicad-libraries:DRILL_NP" (id 2) (at 279.4 156.21 0)
+    (property "Footprint" "kicad-libraries:DRILL_NP_New" (id 2) (at 279.4 156.21 0)
       (effects (font (size 1.524 1.524)) hide)
     )
@@
       (effects (font (size 1.524 1.524)))
     )
-    (property "Footprint" "kicad-libraries:DRILL_NP" (id 2) (at 279.4 161.29 0)
+    (property "Footprint" "kicad-libraries:DRILL_NP_New" (id 2) (at 279.4 161.29 0)
       (effects (font (size 1.524 1.524)) hide)
     )
@@
       (effects (font (size 1.524 1.524)))
     )
-    (property "Footprint" "kicad-libraries:DRILL_NP" (id 2) (at 270.51 161.29 0)
+    (property "Footprint" "kicad-libraries:DRILL_NP_New" (id 2) (at 270.51 161.29 0)
       (effects (font (size 1.524 1.524)) hide)
     )
@@
       (effects (font (size 1.524 1.524)))
     )
-    (property "Footprint" "kicad-libraries:DRILL_NP" (id 2) (at 270.51 156.21 0)
+    (property "Footprint" "kicad-libraries:DRILL_NP_New" (id 2) (at 270.51 156.21 0)
       (effects (font (size 1.524 1.524)) hide)
     )
@@
     )
     (path "/00000000-0000-0000-0000-00004c6050a5"
-      (reference "U4") (unit 1) (value "DRILL") (footprint "kicad-libraries:DRILL_NP")
+      (reference "U4") (unit 1) (value "DRILL") (footprint "kicad-libraries:DRILL_NP_New")
     )
     (path "/00000000-0000-0000-0000-00004c6050a2"
-      (reference "U5") (unit 1) (value "DRILL") (footprint "kicad-libraries:DRILL_NP")
+      (reference "U5") (unit 1) (value "DRILL") (footprint "kicad-libraries:DRILL_NP_New")
     )
     (path "/00000000-0000-0000-0000-00004c605099"
-      (reference "U6") (unit 1) (value "DRILL") (footprint "kicad-libraries:DRILL_NP")
+      (reference "U6") (unit 1) (value "DRILL") (footprint "kicad-libraries:DRILL_NP_New")
     )
     (path "/00000000-0000-0000-0000-00004c60509f"
-      (reference "U7") (unit 1) (value "DRILL") (footprint "kicad-libraries:DRILL_NP")
-    )
-  )
+      (reference "U7") (unit 1) (value "DRILL") (footprint "kicad-libraries:DRILL_NP_New")
+    )
+  )

Commit message: Data Cleanup
Parts:
- U4, U5, U6, U7: footprint kicad-libraries:DRILL_NP_New -> kicad-libraries:DRILL_NP
Changed lines of the file:
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@@
       (effects (font (size 1.524 1.524)))
     )
-    (property "Footprint" "kicad-libraries:DRILL_NP_New" (id 2) (at 279.4 156.21 0)
+    (property "Footprint" "kicad-libraries:DRILL_NP" (id 2) (at 279.4 156.21 0)
       (effects (font (size 1.524 1.524)) hide)
     )
@@
       (effects (font (size 1.524 1.524)))
     )
-    (property "Footprint" "kicad-libraries:DRILL_NP_New" (id 2) (at 279.4 161.29 0)
+    (property "Footprint" "kicad-libraries:DRILL_NP" (id 2) (at 279.4 161.29 0)
       (effects (font (size 1.524 1.524)) hide)
     )
@@
       (effects (font (size 1.524 1.524)))
     )
-    (property "Footprint" "kicad-libraries:DRILL_NP_New" (id 2) (at 270.51 161.29 0)
+    (property "Footprint" "kicad-libraries:DRILL_NP" (id 2) (at 270.51 161.29 0)
       (effects (font (size 1.524 1.524)) hide)
     )
@@
       (effects (font (size 1.524 1.524)))
     )
-    (property "Footprint" "kicad-libraries:DRILL_NP_New" (id 2) (at 270.51 156.21 0)
+    (property "Footprint" "kicad-libraries:DRILL_NP" (id 2) (at 270.51 156.21 0)
       (effects (font (size 1.524 1.524)) hide)
     )
@@
     )
     (path "/00000000-0000-0000-0000-00004c6050a5"
-      (reference "U4") (unit 1) (value "DRILL") (footprint "kicad-libraries:DRILL_NP_New")
+      (reference "U4") (unit 1) (value "DRILL") (footprint "kicad-libraries:DRILL_NP")
     )
     (path "/00000000-0000-0000-0000-00004c6050a2"
-      (reference "U5") (unit 1) (value "DRILL") (footprint "kicad-libraries:DRILL_NP_New")
+      (reference "U5") (unit 1) (value "DRILL") (footprint "kicad-libraries:DRILL_NP")
     )
     (path "/00000000-0000-0000-0000-00004c605099"
-      (reference "U6") (unit 1) (value "DRILL") (footprint "kicad-libraries:DRILL_NP_New")
+      (reference "U6") (unit 1) (value "DRILL") (footprint "kicad-libraries:DRILL_NP")
     )
     (path "/00000000-0000-0000-0000-00004c60509f"
-      (reference "U7") (unit 1) (value "DRILL") (footprint "kicad-libraries:DRILL_NP_New")
-    )
-  )
+      (reference "U7") (unit 1) (value "DRILL") (footprint "kicad-libraries:DRILL_NP")
+    )
+  )
