File: hardware/industrial-dual-relay.kicad_sch (KiCad schematic)
At the start: 27 parts, among them P1 CON-SENSOR2, P2 BOOT, P3 CONN_8, P4 Debug, Q1 SSM6N7002KFU, Q2 G5Q-1, Q3 G5Q-1, U1 XMC1100, U4 DRILL, U5 DRILL, U6 DRILL, U7 DRILL

Commit message: version 1.3: fix dates and pcb rotation
Other:
- note added: "Copyright Tinkerforge GmbH 2026. This documentation describes Open Hardware and is licensed under the CERN OHL v. 1.1. You may redistribute and modify this documentation under the terms of the CERN OHL v.1.1. (http://ohwr.org/cernohl). This documentation is distributed WITHOUT ANY EXPRESS OR IMPLIED WARRANTY, INCLUDING OF MERCHANTABILITY, SATISFACTORY QUALITY AND FITNESS FOR A PARTICULAR PURPOSE.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"
- note removed: "Copyright Tinkerforge GmbH 2023. This documentation describes Open Hardware and is licensed under the CERN OHL v. 1.1. You may redistribute and modify this documentation under the terms of the CERN OHL v.1.1. (http://ohwr.org/cernohl). This documentation is distributed WITHOUT ANY EXPRESS OR IMPLIED WARRANTY, INCLUDING OF MERCHANTABILITY, SATISFACTORY QUALITY AND FITNESS FOR A PARTICULAR PURPOSE.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"
Changed lines of the file:
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@@
 	(title_block
 		(title "Industrial Dual Relay")
-		(date "2023-01-24")
-		(rev "1.2")
+		(date "2026-09-16")
+		(rev "1.3")
 		(company "Tinkerforge GmbH")
 		(comment 1 "Licensed under CERN OHL v.1.1")
-		(comment 2 "Copyright (©) 2023, B.Nordmeyer <bastian@tinkerforge.com>")
+		(comment 2 "Copyright (©) 2026, B.Nordmeyer <bastian@tinkerforge.com>")
 	)
-	(text "Copyright Tinkerforge GmbH 2023.\nThis documentation describes Open Hardware and is licensed under the\nCERN OHL v. 1.1.\nYou may redistribute and modify this documentation under the terms of the\nCERN OHL v.1.1. (http://ohwr.org/cernohl). This documentation is distributed\nWITHOUT ANY EXPRESS OR IMPLIED WARRANTY, INCLUDING OF\nMERCHANTABILITY, SATISFACTORY QUALITY AND FITNESS FOR A\nPARTICULAR PURPOSE. Please see the CERN OHL v.1.1 for applicable\nconditions\n"
+	(text "Copyright Tinkerforge GmbH 2026.\nThis documentation describes Open Hardware and is licensed under the\nCERN OHL v. 1.1.\nYou may redistribute and modify this documentation under the terms of the\nCERN OHL v.1.1. (http://ohwr.org/cernohl). This documentation is distributed\nWITHOUT ANY EXPRESS OR IMPLIED WARRANTY, INCLUDING OF\nMERCHANTABILITY, SATISFACTORY QUALITY AND FITNESS FOR A\nPARTICULAR PURPOSE. Please see the CERN OHL v.1.1 for applicable\nconditions\n"
 		(exclude_from_sim no)
 		(at 13.97 195.58 0)
